Commit message: Fix left/right mass and inertia asymmetry in the v2 hands (issue #19, item 3)
The v2 left hand was a separate Fusion360 export rather than a mirror of the
right, so its inertial properties disagreed with the right hand's. Most
visibly the carpals: 0.85426 kg on the left vs 0.13539 kg on the right. The
left carpals mesh was also a stale, different part (109.53 cm3, COM at
x = +4.52 mm) rather than the mirror of the right (119.27 cm3, x = +5.88 mm),
so the left mass was 0.854 kg over 109.5 cm3 -- an implied density of
7800 kg/m3, i.e. steel, where every other link sits at 1000-1220 kg/m3.

Regenerate all 44 left-hand files as the exact sagittal (x=0) mirror of the
right via utils/mirror_left_from_right.py, so left == mirror(right) holds
exactly for URDF, MJCF body and STL geometry. Verified with --check.

This addresses item 3 of issue #19 only. The forearm's steel density (item 1)
and the 1e4 inertia scale error (item 2) are present on BOTH hands equally and
are unaffected by mirroring -- the two hands are now consistent with each
other, and both still carry those errors.

The wrist joint origin is deliberately left untouched: the left now mirrors
whatever the right currently has (roll -0.610865 rad preserved on both), so
this commit makes no change to the wrist rest pose.

Reported-by: martinovzky
Co-Authored-By: Claude Opus 5 (1M context) <noreply@anthropic.com>
Claude-Session: https://claude.ai/code/session_01RPemG2GBp5VQdKs46H7EC1

File: v2/models/urdf/orcahand_left.urdf (robot description, URDF)
Before this commit: robot orcahand_left, 19 links, 18 joints
Links:
- link I-AP-L_57ce92f7: mass 0.004581542163025142 -> 0.004590288233037025
- link L-Carpals_719fff8c: mass 0.8542565487567293 -> 0.13538810897856451
- link L-T-AP_58680c44: mass 0.007005325272888604 -> 0.007004136465100992
- link T-TP-L_92b8100b: mass 0.007979567574495501 -> 0.00797873207561227
Joints:
- joint I-AP-L_57ce92f7_to_L-Carpals_719fff8c: axis -0.03128510081059521 0.16814409541512249 -0.9852658553123104 -> -8.326672684688674e-17 -3.3306690738754696e-16 -0.9999999999999991; limit lower=-0.436332313 upper=0.5235987756 effort=100 velocity=100 -> lower=-0.4363323129985824 upper=0.5235987755982988 effort=100 velocity=100; origin xyz=0.02724097903991439 -0.0022069668041747375 0.06940680269673632 rpy=-1.6539349343007128 1.3875235793993306 -3.137397887644825 -> xyz=0.027240979039914386 -0.002206966804174762 0.06940680269673646 rpy=1.6538568135338134 -1.3873496487488786 0.0042742186040372054
- joint I-FingerTipAssembly_ed91b18a_to_I-PP_3df4f91d: axis -3.552713678800501e-15 -0.9999999999999964 2.706168622523819e-16 -> -3.608224830031759e-15 0.999999999999996 -2.7755575615628914e-16; origin xyz=0.0014999999999999992 -3.8017921562950314e-18 0.03699999999999992 rpy=3.191891195797317e-16 0.0 6.661338147750924e-15 -> xyz=-0.0015000000000000417 -7.819255613844171e-18 0.037000000000000026 rpy=3.3306690738754617e-16 0.0 -6.77236045021344e-15
- joint I-PP_3df4f91d_to_I-AP-L_57ce92f7: axis 5.995204332975845e-15 -1.0000000000000038 2.0816681711721685e-17 -> 5.828670879282072e-15 1.0000000000000036 -1.1102230246251565e-16; origin xyz=-0.01915096815087688 2.189902551977232e-18 -0.0009999999999970408 rpy=0.0 -1.5707963267948903 0.0 -> xyz=0.01915096815087666 -4.499288227880137e-18 -0.0009999999999971549 rpy=-2.9439233600320843e-16 1.570796326794891 0.0
- joint L-Carpals_719fff8c_to_TopTower-Model_4a80d30e: axis -0.9999999999999971 1.767581259681953e-16 -1.318389841742366e-16 -> -0.9999999999999963 1.1270242357758872e-16 -5.94450127715256e-17; origin xyz=4.336808689942018e-19 1.734723475976807e-18 0.04000000000000012 rpy=-0.610865285723758 2.220446049250313e-16 -1.5707963267948992 -> xyz=-5.551115123125783e-17 2.3418766925686896e-17 0.04000000000000006 rpy=-0.610865285723758 0.0 1.5707963267948992
- joint L-T-AP_58680c44_to_T-TP-L_92b8100b: axis 1.27675647831893e-15 0.3420201433256675 -0.9396926207859057 -> -1.4988010832439613e-15 -0.3420201433256641 -0.9396926207859044; origin xyz=-0.008000000000000014 -2.3699749316290387e-17 -0.003850000000000124 rpy=1.2217304763960308 -2.886579864025407e-15 1.9984014443252818e-15 -> xyz=0.007999999999728488 -1.8648424965940806e-17 -0.003850000000000026 rpy=-1.221730476396032 1.9984014443252818e-15 2.3314683517128287e-15
- joint M-AP_6ec59111_to_L-Carpals_719fff8c: axis -0.025208135220825684 -0.17180872948058878 -0.9848077530122064 -> 8.881784197001252e-16 5.551115123125783e-17 -0.9999999999999994; origin xyz=-0.015307722147416563 -0.0032183646651256395 0.07130479703009845 rpy=1.570796326794893 1.4251136941309301 -0.08726646259971993 -> xyz=-0.015307722147416544 -0.003218364665125601 0.07130479703009855 rpy=-1.5707963267948946 -1.4250613342533707 3.054326190990075
- joint M-AP_e04a96f2_to_L-Carpals_719fff8c: axis -6.106226635438361e-16 1.6653345369377348e-16 -0.9999999999999963 -> 1.1102230246251565e-15 2.220446049250313e-16 -0.9999999999999971; origin xyz=0.005706333727246732 -0.004023404072025596 0.07850189342716873 rpy=-1.5707963267947105 1.5681085197468256 -3.141592653589607 -> xyz=0.005706333727246699 -0.004023404072025678 0.07850189342716887 rpy=1.5707963267946425 -1.5681783329169052 2.544631172440859e-13
- joint M-FingerTipAssembly_34afb748_to_M-PP_08efa608: axis -3.2751579226442118e-15 -0.9999999999999984 7.968885967768458e-17 -> -3.2751579226442118e-15 0.9999999999999977 -4.440892098500626e-16; origin xyz=0.0020000000000000013 -7.514798000251117e-18 0.04000000000000003 rpy=2.3310346708438266e-16 0.0 6.217248937900862e-15 -> xyz=-0.0020000000000000313 -5.598548939047626e-18 0.0400000000000001 rpy=5.551115123125779e-16 -4.440892098500626e-16 -6.550315845288408e-15
- joint M-FingerTipAssembly_424a8e75_to_M-PP_8660a1eb: axis -3.4416913763379853e-15 -0.9999999999999967 1.5265566588595902e-16 -> -2.942091015256665e-15 0.999999999999996 -2.220446049250313e-16; origin xyz=0.0020000000000000026 1.0167803431570436e-17 0.04000000000000024 rpy=2.2204460492503052e-16 0.0 6.550315845288409e-15 -> xyz=-0.0019999999999998678 1.5882195667426256e-18 0.040000000000000126 rpy=2.2204460492503052e-16 0.0 -6.217248937900862e-15
- joint M-PP_08efa608_to_M-AP_e04a96f2: axis 5.773159728050814e-15 -1.000000000000006 -1.476683358925257e-16 -> 6.050715484207103e-15 1.0000000000000058 1.1102230246251565e-16; origin xyz=-0.019866967942905434 2.2433222511080304e-18 -0.000999999999995544 rpy=0.0 -1.5707963267948908 0.0 -> xyz=0.019866967942905277 -1.8423293703642938e-17 -0.0009999999999957202 rpy=0.0 1.5707963267948903 0.0
- joint M-PP_8660a1eb_to_M-AP_6ec59111: axis 6.050715484207103e-15 -1.0000000000000036 -5.551115123125783e-17 -> 5.9396931817445875e-15 1.0000000000000042 -1.1102230246251565e-16; origin xyz=-0.01986696794290542 7.724722121653367e-18 -0.0009999999999955448 rpy=0.0 -1.5707963267948908 0.0 -> xyz=0.01986696794290542 3.8657355141463114e-17 -0.00099999999999545 rpy=0.0 1.5707963267948908 0.0
- joint P-AP_f5e42b61_to_L-Carpals_719fff8c: axis -0.13297994090837154 -0.34829476172536833 -0.927904679517606 -> 9.71445146547012e-16 -1.6653345369377348e-16 -0.9999999999999984; origin xyz=-0.03564171604590434 0.0006891586859576484 0.06205424192069404 rpy=1.5294679618327596 1.2029145266720778 -0.22960913173696929 -> xyz=-0.035641716045904354 0.0006891586859576128 0.06205424192069395 rpy=-1.529473573814961 -1.2028622114983025 2.9119895363116646
- joint P-FingerTipAssembly_cd219176_to_P-PP_1d411b9b: axis -3.164135620181696e-15 -0.9999999999999976 1.1102230246251565e-16 -> -2.609024107869118e-15 0.9999999999999968 -3.885780586188048e-16; origin xyz=0.0009999999999999979 -1.3225694162272767e-17 0.030999999999999892 rpy=1.3877787807814457e-16 0.0 5.884182030513316e-15 -> xyz=-0.000999999999999998 3.208202345938654e-17 0.030999999999999632 rpy=1.1102230246251565e-16 0.0 -6.217248937900863e-15
- joint P-PP_1d411b9b_to_P-AP_f5e42b61: axis 5.495603971894525e-15 -1.0000000000000044 2.7755575615628914e-17 -> 6.439293542825908e-15 1.0000000000000049 -6.661338147750939e-16; origin xyz=-0.01774999999999982 -5.95919845612908e-17 -0.0009999999999999916 rpy=0.0 -1.5707963267948915 0.0 -> xyz=0.017750000000000075 -4.698582746252626e-17 -0.0010000000000000768 rpy=0.0 1.5707963267948908 0.0
- joint T-DP_307db3cc_to_T-PP_ef067304: axis -8.604228440844963e-16 -0.9999999999999971 -4.440892098500626e-16 -> 4.718447854656915e-16 0.9999999999999946 -3.164135620181696e-15; origin xyz=0.0010000000000000896 -1.3141266374808417e-17 0.03200000000000025 rpy=0.0 0.0 3.885780586188038e-15 -> xyz=-0.0009999999999999985 1.1880660448999647e-16 0.03200000000000021 rpy=0.0 0.0 3.830269434956779e-15
- joint T-PP_ef067304_to_L-T-AP_58680c44: axis 3.1086244689504383e-15 -1.0000000000000049 -2.7755575615628914e-16 -> -3.1363800445660672e-15 1.0000000000000027 -2.942091015256665e-15; origin xyz=-0.02800000000000005 7.823464669468643e-17 -3.231584414086884e-18 rpy=-3.1415926535897927 1.570796326794893 0.0 -> xyz=0.027999999999999976 4.673366946417151e-18 1.305542026140606e-16 rpy=-3.1415926535897927 -1.5707963267948921 0.0
- joint T-TP-L_92b8100b_to_L-Carpals_719fff8c: axis -2.435551760271437e-15 3.885780586188048e-16 0.9999999999999951 -> -7.771561172376096e-16 -5.412337245047638e-16 0.9999999999999931; origin xyz=0.028398719136200797 0.010997180928709051 0.03058953349163119 rpy=-0.6616685732384568 0.3857244523560657 -1.7091857348501476 -> xyz=0.028398719136200776 0.010997180928709077 0.03058953349163134 rpy=0.6614951404674763 -0.3860568562160207 1.4328677049607634
- joint TopTower-Model_4a80d30e_to_ForeArmStructure-Model_e18f2368: origin xyz=-0.010000000000000018 0.05230000000000584 -2.0816681711721685e-17 rpy=-1.5707963267948966 1.570796326794894 0.0 -> xyz=0.010000000000000018 0.05230000000000584 -2.0816681711721685e-17 rpy=-1.5707963267948966 -1.570796326794894 0.0

Commit message: Remove the spurious -35 deg roll from the v2 wrist joint origins
Both v2 wrist joint origins carried rpy roll = -0.610865285723758 rad, baked
into the URDF by the Fusion360 export. Three independent checks say it is an
export artifact rather than design intent:

  - v1, the known-good shipping model, has wrist rpy = 0.0 0.0 0.0
  - both v2 MJCFs have no roll at all (carpals quat is a pure -90 deg about z)
  - the roll is exactly the wrist's own UPPER joint limit, +0.6108652381980153
    rad = 35.000 deg, matching to 4.8e-08 rad

That last coincidence is the signature of a CAD assembly saved with the wrist
parked at one end of its travel, with the exporter writing that pose into the
joint origin.

It did not break URDF validity, which is why it survived, but it shifted where
q = 0 sits: anything commanding a wrist angle saw the model 35 deg away from
the hardware at the same commanded angle. Rendering both variants at qpos = 0
shows the hand in line with the forearm at roll = 0 and visibly cocked back at
roll = -35 deg.

Set the roll to zero on the right and regenerate the left through
utils/mirror_left_from_right.py so left == mirror(right) still holds exactly
(verified with --check). The v2 URDFs and MJCFs now agree on the wrist rest
pose for the first time.

Supersedes 9fa90c1, which unified the left wrist onto the right's rolled pose
rather than removing the roll from both.

Co-Authored-By: Claude Opus 5 (1M context) <noreply@anthropic.com>
Claude-Session: https://claude.ai/code/session_01RPemG2GBp5VQdKs46H7EC1

File: v2/models/urdf/orcahand_left.urdf (robot description, URDF)
Before this commit: robot orcahand_left, 19 links, 18 joints
Joints:
- joint L-Carpals_719fff8c_to_TopTower-Model_4a80d30e: origin xyz=-5.551115123125783e-17 2.3418766925686896e-17 0.04000000000000006 rpy=-0.610865285723758 0.0 1.5707963267948992 -> xyz=-5.551115123125783e-17 2.3418766925686896e-17 0.04000000000000006 rpy=0.0 0.0 1.5707963267948992
