Commit message: vKTH model with this hand's calibrated joint limits

File: v1/models/urdf/orcahand_right.urdf (robot description, URDF)
Before this commit: robot orcahand_right, 42 links, 41 joints
Joints:
- joint right_thumb_mcp: limit lower=-0.87266 upper=0.87266 effort=100 velocity=100 -> lower=-1.48353 upper=0.87266 effort=100 velocity=100

File: vKTH/models/urdf/orcahand_right.urdf (robot description, URDF)
Before this commit: robot orcahand_right, 19 links, 18 joints
Joints:
- joint I-AP-R_d95d02d1_to_R-Carpals_8d1f1041: limit lower=-0.4363323129985824 upper=0.5235987755982988 effort=100 velocity=100 -> lower=-0.5235987755982988 upper=0.5235987755982988 effort=100 velocity=100
- joint I-PP_bacbd481_to_I-AP-R_d95d02d1: limit lower=-0.4363323129985824 upper=1.7453292519943295 effort=100 velocity=100 -> lower=-1.0471975511965976 upper=1.7453292519943295 effort=100 velocity=100
- joint M-AP_6ec59111_to_R-Carpals_8d1f1041: limit lower=-0.47123889803846897 upper=0.47123889803846897 effort=100 velocity=100 -> lower=-0.5235987755982988 upper=0.5235987755982988 effort=100 velocity=100
- joint M-AP_e04a96f2_to_R-Carpals_8d1f1041: limit lower=-0.47123889803846897 upper=0.47123889803846897 effort=100 velocity=100 -> lower=-0.5235987755982988 upper=0.5235987755982988 effort=100 velocity=100
- joint M-FingerTipAssembly_34afb748_to_M-PP_08efa608: limit lower=-0.2617993877991494 upper=1.8675022996339325 effort=100 velocity=100 -> lower=-0.3490658503988659 upper=1.8675022996339325 effort=100 velocity=100
- joint M-PP_08efa608_to_M-AP_e04a96f2: limit lower=-0.4363323129985824 upper=1.7453292519943295 effort=100 velocity=100 -> lower=-1.0471975511965976 upper=1.7453292519943295 effort=100 velocity=100
- joint M-PP_8660a1eb_to_M-AP_6ec59111: limit lower=-0.4363323129985824 upper=1.7453292519943295 effort=100 velocity=100 -> lower=-1.0471975511965976 upper=1.7453292519943295 effort=100 velocity=100
- joint P-FingerTipAssembly_cd219176_to_P-PP_1d411b9b: limit lower=-0.2617993877991494 upper=1.8675022996339325 effort=100 velocity=100 -> lower=-0.2617993877991494 upper=1.8849555921538759 effort=100 velocity=100
- joint P-PP_1d411b9b_to_P-AP_f5e42b61: limit lower=-0.4363323129985824 upper=1.7453292519943295 effort=100 velocity=100 -> lower=-1.0471975511965976 upper=1.7453292519943295 effort=100 velocity=100
- joint R-T-AP_a9723101_to_T-TP-R_1c2b802d: limit lower=-0.3141592653589793 upper=0.9599310885968813 effort=100 velocity=100 -> lower=-0.2792526803190927 upper=0.6981317007977318 effort=100 velocity=100
- joint T-DP_b7429e50_to_T-PP_68395e98: limit lower=-0.2617993877991494 upper=1.8675022996339325 effort=100 velocity=100 -> lower=-0.9599310885968813 upper=1.8675022996339325 effort=100 velocity=100
- joint T-PP_68395e98_to_R-T-AP_a9723101: limit lower=-0.4363323129985824 upper=1.7453292519943295 effort=100 velocity=100 -> lower=-1.1693705988362009 upper=1.5707963267948966 effort=100 velocity=100
- joint T-TP-R_1c2b802d_to_R-Carpals_8d1f1041: limit lower=-1.0472 upper=0.5759586531581288 effort=100 velocity=100 -> lower=-0.7504915783575618 upper=0.8203047484373349 effort=100 velocity=100
